File: hardware/usb-current-meter-8x.sch (EAGLE design)
At the start: 35 parts, among them IC3 MEGA48/88/168-AU, IC9 OPA2234U, X7 MC2

Commit message: hardware: first version with 1 module
Parts:
- added H1, H2, H3, H4: MOUNT-PAD-ROUND3.2, holes:MOUNT-PAD-ROUND3.2
Connections:
- removed net SC_OUT: C40.1, C41.1, C43.1, R60.2
- net GND: now also H1.MOUNT, H2.MOUNT, H3.MOUNT, H4.MOUNT
- net IN_CH0: now also C40.1, C41.1, C43.1, R60.2

Commit message: hardware: progress save
Parts:
- added C14, C17, C19, C22, C27, C29, C4, C7: 100n, rcl:C-EUC0805
- added C15, C16, C18, C20, C21, C23, C25, C26, C28, C5, C6, C8: 1u, rcl:C-EUC0805
- added D1, D2, D3, D4: BAT54, diode:BAT54
- added IC2, IC4, IC5, IC6: OPA2234U, burr-brown:OPA2234U
- added R10, R14, R15, R16, R17, R18, R19, R22, R23, R24, R25, R26, R27, R30, R31, R32, R33, R42, R43, R5, R6, R7, R8, R9: tbd, rcl:R-EU_R0603
- added R11, R20, R28, R36: 100k, rcl:R-EU_R0603
- added R12, R21, R29, R37, R4: Rload, rcl:R-EU_R0805
- added X1, X2, X3, X4, X5: MC2, con-phoenix-381_l:MC2
Connections:
- net SC_IN_B renamed SC_IN_B_0
- removed net SC_IN_A: R53.2, R54.1, X7.1.SK
- new net N$10: IC2B.-IN, R7.2, R8.1
- new net N$11: IC2B.OUT, R11.1, R8.2
- new net N$12: IC4A.-IN, R14.2, R15.1
- new net N$13: D2.A, IC4A.OUT
- new net N$14: D2.C, IC4B.+IN, R15.2
- new net N$15: IC4B.-IN, R16.2, R17.1
- new net N$16: IC4B.OUT, R17.2, R20.1
- new net N$17: IC6A.-IN, R30.2, R31.1
- new net N$18: D4.A, IC6A.OUT
- new net N$19: D4.C, IC6B.+IN, R31.2
- new net N$20: IC6B.-IN, R32.2, R33.1
- new net N$21: IC6B.OUT, R33.2, R36.1
- new net N$22: IC5A.-IN, R22.2, R23.1
- new net N$23: D3.A, IC5A.OUT
- new net N$24: D3.C, IC5B.+IN, R23.2
- new net N$25: IC5B.-IN, R24.2, R25.1
- new net N$26: IC5B.OUT, R25.2, R28.1
- new net N$7: IC2A.-IN, R5.2, R6.1
- new net N$8: D1.A, IC2A.OUT
- new net N$9: D1.C, IC2B.+IN, R6.2
- new net SC_IN_A_0: R29.2, R30.1, R53.2, R54.1, X4.1.SK, X7.1.SK
- new net SC_IN_A_1: R4.2, R5.1, X1.1.SK
- new net SC_IN_A_2: R12.2, R14.1, X2.1.SK
- new net SC_IN_A_3: R21.2, R22.1, X3.1.SK
- new net SC_IN_B_1: C4.1, R10.2, R4.1, R9.1, X1.2.SK
- new net SC_IN_B_2: C14.1, R12.1, R18.1, R19.2, X2.2.SK
- new net SC_IN_B_3: C19.1, R21.1, R26.1, R27.2, X3.2.SK
- new net SC_IN_B_5: C29.1, R37.1, R42.1, R43.2, X5.2.SK
- net GND: now also C14.2, C15.2, C16.2, C17.2, C18.2, C19.2, C20.2, C21.2, C22.2, C23.2, C25.2, C26.2, C27.2, C28.2, C29.2, C4.2, C5.2, C6.2, C7.2, C8.2, IC2A.+IN, IC2A.V-, IC4A.+IN, IC4A.V-, IC5A.+IN, IC5A.V-, IC6A.+IN, IC6A.V-, R10.1, R16.1, R19.1, R24.1, R27.1, R29.1, R32.1, R43.1, R7.1, X4.2.SK
- net IN_CH0: now also C25.1, C26.1, C28.1, R36.2
- net IN_CH1: now also C5.1, C6.1, C8.1, R11.2, R37.2, X5.1.SK
- net IN_CH2: now also C15.1, C16.1, C18.1, R20.2
- net IN_CH3: now also C20.1, C21.1, C23.1, R28.2
- net VCC: now also C17.1, C22.1, C27.1, C7.1, IC2A.V+, IC4A.V+, IC5A.V+, IC6A.V+, R18.2, R26.2, R42.2, R9.2
Other:
- note added: "Channel 1"
- note added: "Channel 2"
- note added: "Channel 3"

Commit message: hardware: 8x schematic updated
Parts:
- removed C14, C17, C19, C22, C27, C29, C39, C7: 100n, rcl:C-EUC0805
- removed C15, C16, C18, C20, C21, C23, C25, C26, C28, C6, C8: 1u, rcl:C-EUC0805
- removed D1, D2, D3, D4: BAT54, diode:BAT54
- removed IC2, IC4, IC5, IC6: OPA2234U, burr-brown:OPA2234U
- removed JP1: (no value), SparkFun:M04PTH
- removed R10, R14, R15, R16, R17, R18, R19, R22, R23, R24, R25, R26, R27, R30, R31, R32, R33, R42, R43, R5, R58, R59, R6, R7, R8, R9: tbd, rcl:R-EU_R0603
- removed R11, R20, R28, R36: 100k, rcl:R-EU_R0603
- removed R12, R21, R29, R37: Rload, rcl:R-EU_R0805
- removed X1, X2, X3, X4, X5: MC2, con-phoenix-381_l:MC2
- C5: value 1u -> 100n
- R4: value Rload -> tbd; device rcl:R-EU_R0805 -> rcl:R-EU_R0603
Connections:
- net IN_CH4 renamed CH4
- net IN_CH5 renamed CH5
- net IN_CH6 renamed CH6
- net IN_CH7 renamed CH7
- removed net IN_CH0: C25.1, C26.1, C28.1, C40.1, C41.1, C43.1, IC3.PC0(ADC0/PCINT8), R36.2, R60.2
- removed net IN_CH1: C5.1, C6.1, C8.1, IC3.PC1(ADC1/PCINT9), R11.2, R37.2, X5.1.SK
- removed net IN_CH2: C15.1, C16.1, C18.1, IC3.PC2(ADC2/PCINT10), R20.2
- removed net IN_CH3: C20.1, C21.1, C23.1, IC3.PC3(ADC3/PCINT11), R28.2
- removed net N$10: IC2B.-IN, R7.2, R8.1
- removed net N$11: IC2B.OUT, R11.1, R8.2
- removed net N$12: IC4A.-IN, R14.2, R15.1
- removed net N$13: D2.A, IC4A.OUT
- removed net N$14: D2.C, IC4B.+IN, R15.2
- removed net N$15: IC4B.-IN, R16.2, R17.1
- removed net N$16: IC4B.OUT, R17.2, R20.1
- removed net N$17: IC6A.-IN, R30.2, R31.1
- removed net N$18: D4.A, IC6A.OUT
- removed net N$19: D4.C, IC6B.+IN, R31.2
- removed net N$20: IC6B.-IN, R32.2, R33.1
- removed net N$21: IC6B.OUT, R33.2, R36.1
- removed net N$22: IC5A.-IN, R22.2, R23.1
- removed net N$23: D3.A, IC5A.OUT
- removed net N$24: D3.C, IC5B.+IN, R23.2
- removed net N$25: IC5B.-IN, R24.2, R25.1
- removed net N$26: IC5B.OUT, R25.2, R28.1
- removed net N$8: D1.A, IC2A.OUT
- removed net N$9: D1.C, IC2B.+IN, R6.2
- removed net SC_IN_A_0: R29.2, R30.1, R53.2, R54.1, X4.1.SK, X7.1.SK
- removed net SC_IN_A_1: R4.2, R5.1, X1.1.SK
- removed net SC_IN_A_2: R12.2, R14.1, X2.1.SK
- removed net SC_IN_A_3: R21.2, R22.1, X3.1.SK
- removed net SC_IN_B_0: C39.1, R53.1, R58.1, R59.2, X7.2.SK
- removed net SC_IN_B_1: C4.1, R10.2, R4.1, R9.1, X1.2.SK
- removed net SC_IN_B_2: C14.1, R12.1, R18.1, R19.2, X2.2.SK
- removed net SC_IN_B_3: C19.1, R21.1, R26.1, R27.2, X3.2.SK
- removed net SC_IN_B_5: C29.1, R37.1, R42.1, R43.2, X5.2.SK
- removed net UART_RX: IC3.PD0(RXD/PCINT16), JP1.3
- removed net UART_TX: IC3.PD1(TXD/PCINT17), JP1.2
- new net CH0: C40.1, C41.1, C43.1, IC3.PC0(ADC0/PCINT8), R60.2
- new net CH0_GAIN: IC3.PD0(RXD/PCINT16), R4.1, R56.2
- new net CH0_IN: C4.1, R53.2, R54.1, X7.1.SK
- new net CH1: IC3.PC1(ADC1/PCINT9)
- new net CH1_GAIN: IC3.PD1(TXD/PCINT17)
- new net CH2: IC3.PC2(ADC2/PCINT10)
- new net CH2_GAIN: IC3.PD5(T1/OC0B/PCINT21)
- new net CH3: IC3.PC3(ADC3/PCINT11)
- new net CH3_GAIN: IC3.PD6(AIN0/OC0A/PCINT22)
- new net CH4_GAIN: IC3.PD7(AIN1/PCINT23)
- new net CH5_GAIN: IC3.PB0(ICP1/CLKO/PCINT0)
- new net CH6_GAIN: IC3.PB1(OC1A/PCINT1)
- new net CH7_GAIN: IC3.PB2(SS/OC1B/PCINT2)
- net GND: now also R53.1, X7.2.SK; no longer C14.2, C15.2, C16.2, C17.2, C18.2, C19.2, C20.2, C21.2, C22.2, C23.2, C25.2, C26.2, C27.2, C28.2, C29.2, C39.2, C5.2, C6.2, C7.2, C8.2, IC2A.+IN, IC2A.V-, IC4A.+IN, IC4A.V-, IC5A.+IN, IC5A.V-, IC6A.+IN, IC6A.V-, JP1.1, R10.1, R16.1, R19.1, R24.1, R27.1, R29.1, R32.1, R43.1, R59.1, R7.1, X4.2.SK
- net LED: now also IC3.PD3(INT1/OC2B/PCINT19); no longer IC3.PB0(ICP1/CLKO/PCINT0)
- net N$40: now also C5.1; no longer R56.2
- net N$7: now also C5.2, R4.2; no longer IC2A.-IN, R5.2, R6.1
- net VCC: no longer C17.1, C22.1, C27.1, C7.1, IC2A.V+, IC4A.V+, IC5A.V+, IC6A.V+, JP1.4, R18.2, R26.2, R42.2, R58.2, R9.2
Other:
- note removed: "Channel 1"
- note removed: "Channel 2"
- note removed: "Channel 3"
- note removed: "UART"
- moved on the sheet: C4, C40, C41, C42, C43, C5, D7, IC9A, IC9B, R4, R53, R54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

Commit message: 8x: progress save
Parts:
- added JP1: (no value), SparkFun-Connectors:M04PTH
- added U$2: Fabio Baltieri, balto:CREATIVE_COMMONS
Connections:
- new net RX: JP1.3
- new net TX: JP1.2
- net GND: now also JP1.1
- net VCC: now also JP1.4
Other:
- note added: "UART"
Changed lines of the file:
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@@
 <part name="R4" library="rcl" deviceset="R-EU_" device="R0603" value="tbd"/>
 <part name="C5" library="rcl" deviceset="C-EU" device="C0805" value="100n"/>
+<part name="U$2" library="balto" deviceset="CREATIVE_COMMONS" device="" value="Fabio Baltieri"/>
+<part name="LICENSE1" library="balto" deviceset="CC_BY-SA" device=""/>
+<part name="JP1" library="SparkFun-Connectors" deviceset="M04" device="PTH"/>
+<part name="P+6" library="supply1" deviceset="VCC" device=""/>
+<part name="GND7" library="supply1" deviceset="GND" device=""/>
 </parts>
 <sheets>
@@
 <wire x1="30.48" y1="106.68" x2="30.48" y2="66.04" width="0.1524" layer="97"/>
 <wire x1="30.48" y1="66.04" x2="10.16" y2="66.04" width="0.1524" layer="97"/>
+<text x="213.36" y="167.64" size="5.08" layer="97">UART</text>
+<wire x1="210.82" y1="175.26" x2="233.68" y2="175.26" width="0.1524" layer="97"/>
+<wire x1="233.68" y1="175.26" x2="233.68" y2="134.62" width="0.1524" layer="97"/>
+<wire x1="233.68" y1="134.62" x2="210.82" y2="134.62" width="0.1524" layer="97"/>
+<wire x1="210.82" y1="134.62" x2="210.82" y2="175.26" width="0.1524" layer="97"/>
 </plain>
 <instances>
@@
 </instance>
 <instance part="C5" gate="G$1" x="337.82" y="223.52"/>
+<instance part="U$2" gate="G$1" x="584.2" y="25.4"/>
+<instance part="LICENSE1" gate="G$1" x="556.26" y="25.4"/>
+<instance part="JP1" gate="G$1" x="226.06" y="149.86" rot="MR0"/>
+<instance part="P+6" gate="VCC" x="218.44" y="160.02"/>
+<instance part="GND7" gate="1" x="218.44" y="142.24"/>
 </instances>
 <busses>
@@
 <wire x1="337.82" y1="205.74" x2="337.82" y2="200.66" width="0.1524" layer="91"/>
 </segment>
+<segment>
+<pinref part="JP1" gate="G$1" pin="1"/>
+<pinref part="GND7" gate="1" pin="GND"/>
+<wire x1="220.98" y1="147.32" x2="218.44" y2="147.32" width="0.1524" layer="91"/>
+<wire x1="218.44" y1="147.32" x2="218.44" y2="144.78" width="0.1524" layer="91"/>
+</segment>
 </net>
 <net name="N$1" class="0">
@@
 <pinref part="C42" gate="G$1" pin="1"/>
 <wire x1="327.66" y1="213.36" x2="327.66" y2="210.82" width="0.1524" layer="91"/>
+</segment>
+<segment>
+<pinref part="JP1" gate="G$1" pin="4"/>
+<pinref part="P+6" gate="VCC" pin="VCC"/>
+<wire x1="220.98" y1="154.94" x2="218.44" y2="154.94" width="0.1524" layer="91"/>
+<wire x1="218.44" y1="154.94" x2="218.44" y2="157.48" width="0.1524" layer="91"/>
 </segment>
 </net>
@@
 </segment>
 </net>
+<net name="TX" class="0">
+<segment>
+<pinref part="JP1" gate="G$1" pin="2"/>
+<wire x1="220.98" y1="149.86" x2="213.36" y2="149.86" width="0.1524" layer="91"/>
+<label x="213.36" y="149.86" size="1.778" layer="95"/>
+</segment>
+</net>
+<net name="RX" class="0">
+<segment>
+<pinref part="JP1" gate="G$1" pin="3"/>
+<wire x1="220.98" y1="152.4" x2="213.36" y2="152.4" width="0.1524" layer="91"/>
+<label x="213.36" y="152.4" size="1.778" layer="95"/>
+</segment>
+</net>

Commit message: 8x: progress save
Parts:
- added C14, C17, C18, C20, C23, C24, C26, C29, C30, C32, C35, C36, C38, C45, C46, C48, C51, C52, C54, C6, C7: 1u, rcl:C-EUC0805
- added C15, C19, C21, C25, C27, C31, C33, C37, C39, C47, C49, C53, C55, C8: 100n, rcl:C-EUC0805
- added C16, C22, C28, C34, C44, C50, C56: 0, rcl:C-EUC0805
- added C57: .1u, rcl:C-EUC0805
- added D1, D2, D3, D4, D5, D6, D8: BAT54, diode:BAT54
- added IC10, IC2, IC4, IC5, IC6, IC7, IC8: OPA2234U, burr-brown:OPA2234U
- added IC12: LTC485S, linear-technology:LTC485S
- added JP2: (no value), SparkFun-Connectors:M02PTH
- added R10, R18, R25, R32, R39, R46, R58: 100k, rcl:R-EU_R0603
- added R11, R19, R26, R33, R40, R47, R59: Rh, rcl:R-EU_R0603
- added R12, R20, R27, R34, R41, R48, R5: Rload, rcl:R-EU_R0805
- added R14, R15, R21, R22, R28, R29, R35, R36, R42, R43, R49, R50, R6, R7: 10k, rcl:R-EU_R0603
- added R16, R23, R30, R37, R44, R51, R8: Rl, rcl:R-EU_R0603
- added R17, R24, R31, R38, R45, R52, R9: Rx, rcl:R-EU_R0603
- added R61: 120, rcl:R-EU_R0603
- added U3: RJ45-8PTH, SparkFun-Connectors:RJ45-8PTH
- added X1, X2, X3, X4, X5, X6, X8: MC2, con-phoenix-381_l:MC2
- C12, C13, C3, C9: value 100n -> .1u
- C5: value 100n -> 0
- R4: value tbd -> Rh
- R54, R55: value tbd -> 10k
- R56: value tbd -> Rl
- R57: value tbd -> Rx
Connections:
- removed net MISO: IC3.PB4(MISO/PCINT4), ISP1.1
- removed net MOSI: IC3.PB3(MOSI/OC2A/PCINT3), ISP1.4
- removed net RX: JP1.3
- removed net SCK: IC3.PB5(SCK/PCINT5), ISP1.3
- removed net TX: JP1.2
- new net 485_N: IC12.B, R61.1, U3.2
- new net 485_P: IC12.A, R61.2, U3.1
- new net CH0_IN1: C15.1, R5.2, R6.1, X1.1.SK
- new net CH0_IN2: C21.1, R12.2, R14.1, X2.1.SK
- new net CH0_IN3: C33.1, R27.2, R28.1, X4.1.SK
- new net CH0_IN4: C39.1, R34.2, R35.1, X5.1.SK
- new net CH0_IN5: C55.1, R48.2, R49.1, X8.1.SK
- new net CH0_IN6: C27.1, R20.2, R21.1, X3.1.SK
- new net CH0_IN8: C49.1, R41.2, R42.1, X6.1.SK
- new net N$10: D1.C, IC2B.+IN, R7.2
- new net N$11: C16.1, IC2B.-IN, R9.1
- new net N$12: IC2B.OUT, R10.1, R9.2
- new net N$13: C16.2, R11.2
- new net N$14: IC4A.-IN, R14.2, R15.1
- new net N$15: D2.A, IC4A.OUT
- new net N$16: D2.C, IC4B.+IN, R15.2
- new net N$17: C22.1, IC4B.-IN, R17.1
- new net N$18: IC4B.OUT, R17.2, R18.1
- new net N$19: C22.2, R19.2
- new net N$20: IC6A.-IN, R28.2, R29.1
- new net N$21: D4.A, IC6A.OUT
- new net N$22: D4.C, IC6B.+IN, R29.2
- new net N$23: C34.1, IC6B.-IN, R31.1
- new net N$24: IC6B.OUT, R31.2, R32.1
- new net N$25: C34.2, R33.2
- new net N$26: IC7A.-IN, R35.2, R36.1
- new net N$27: D5.A, IC7A.OUT
- new net N$28: D5.C, IC7B.+IN, R36.2
- new net N$29: C44.1, IC7B.-IN, R38.1
- new net N$30: IC7B.OUT, R38.2, R39.1
- new net N$31: C44.2, R40.2
- new net N$32: IC10A.-IN, R49.2, R50.1
- new net N$33: D8.A, IC10A.OUT
- new net N$34: D8.C, IC10B.+IN, R50.2
- new net N$35: C56.1, IC10B.-IN, R52.1
- new net N$36: IC10B.OUT, R52.2, R58.1
- new net N$42: C56.2, R59.2
- new net N$43: IC5A.-IN, R21.2, R22.1
- new net N$44: D3.A, IC5A.OUT
- new net N$45: D3.C, IC5B.+IN, R22.2
- new net N$46: C28.1, IC5B.-IN, R24.1
- new net N$47: IC5B.OUT, R24.2, R25.1
- new net N$48: C28.2, R26.2
- new net N$49: IC12.RO, JP2.2
- new net N$55: IC8A.-IN, R42.2, R43.1
- new net N$56: D6.A, IC8A.OUT
- new net N$57: D6.C, IC8B.+IN, R43.2
- new net N$58: C50.1, IC8B.-IN, R45.1
- new net N$59: IC8B.OUT, R45.2, R46.1
- new net N$60: C50.2, R47.2
- new net N$8: IC2A.-IN, R6.2, R7.1
- new net N$9: D1.A, IC2A.OUT
- new net UART_EN: IC12.!RE, IC12.DE, IC3.PD3(INT1/OC2B/PCINT19), ISP1.3
- new net UART_RX: IC3.PD0(RXD/PCINT16), JP1.3, JP2.1
- new net UART_TX: IC12.DI, IC3.PD1(TXD/PCINT17), JP1.2
- net +5V: now also U3.4, U3.5
- net CH0: now also IC3.PC5(ADC5/SCL/PCINT13); no longer IC3.PC0(ADC0/PCINT8)
- net CH0_GAIN: now also IC3.PB4(MISO/PCINT4), ISP1.1; no longer IC3.PD0(RXD/PCINT16)
- net CH1: now also C14.1, C6.1, C7.1, IC3.PC4(ADC4/SDA/PCINT12), R10.2; no longer IC3.PC1(ADC1/PCINT9)
- net CH1_GAIN: now also IC3.PB5(SCK/PCINT5), ISP1.4, R11.1, R8.2; no longer IC3.PD1(TXD/PCINT17)
- net CH2: now also C17.1, C18.1, C20.1, IC3.PC3(ADC3/PCINT11), R18.2; no longer IC3.PC2(ADC2/PCINT10)
- net CH2_GAIN: now also R16.2, R19.1
- net CH3: now also C23.1, C24.1, C26.1, IC3.PC2(ADC2/PCINT10), R25.2; no longer IC3.PC3(ADC3/PCINT11)
- net CH3_GAIN: now also R23.2, R26.1
- net CH4: now also C29.1, C30.1, C32.1, IC3.PC1(ADC1/PCINT9), R32.2; no longer IC3.PC4(ADC4/SDA/PCINT12)
- net CH4_GAIN: now also R30.2, R33.1
- net CH5: now also C35.1, C36.1, C38.1, IC3.PC0(ADC0/PCINT8), R39.2; no longer IC3.PC5(ADC5/SCL/PCINT13)
- net CH5_GAIN: now also R37.2, R40.1
- net CH6: now also C45.1, C46.1, C48.1, IC3.ADC7, R46.2; no longer IC3.ADC6
- net CH6_GAIN: now also R44.2, R47.1
- net CH7: now also C51.1, C52.1, C54.1, IC3.ADC6, R58.2; no longer IC3.ADC7
- net CH7_GAIN: now also R51.2, R59.1
- net GND: now also C14.2, C15.2, C17.2, C18.2, C19.2, C20.2, C21.2, C23.2, C24.2, C25.2, C26.2, C27.2, C29.2, C30.2, C31.2, C32.2, C33.2, C35.2, C36.2, C37.2, C38.2, C39.2, C45.2, C46.2, C47.2, C48.2, C49.2, C51.2, C52.2, C53.2, C54.2, C55.2, C57.2, C6.2, C7.2, C8.2, IC10A.+IN, IC10A.V-, IC12.GND, IC2A.+IN, IC2A.V-, IC4A.+IN, IC4A.V-, IC5A.+IN, IC5A.V-, IC6A.+IN, IC6A.V-, IC7A.+IN, IC7A.V-, IC8A.+IN, IC8A.V-, R12.1, R16.1, R20.1, R23.1, R27.1, R30.1, R34.1, R37.1, R41.1, R44.1, R48.1, R5.1, R51.1, R8.1, U3.7, U3.8, X1.2.SK, X2.2.SK, X3.2.SK, X4.2.SK, X5.2.SK, X6.2.SK, X8.2.SK
- net LED: now also IC3.PB3(MOSI/OC2A/PCINT3); no longer IC3.PD3(INT1/OC2B/PCINT19)
- net VCC: now also C19.1, C25.1, C31.1, C37.1, C47.1, C53.1, C57.1, C8.1, IC10A.V+, IC12.VCC, IC2A.V+, IC4A.V+, IC5A.V+, IC6A.V+, IC7A.V+, IC8A.V+
Other:
- note added: "485"
- note added: "CH0"
- note added: "CH1"
- note added: "CH2"
- note added: "CH3"
- note added: "CH4"
- note added: "CH5"
- note added: "CH6"
- note added: "CH7"
- note removed: "Channel 0"
- moved on the sheet: C1, C10, C11, C12, C13, C2, C3, C4, C40, C41, C42, C43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

Commit message: 8x: progress save
Parts:
- removed H1, H2, H3, H4: MOUNT-PAD-ROUND3.2, holes:MOUNT-PAD-ROUND3.2
- added BOX1: HAMMOND-BOX-XXA, hammond:HAMMOND-BOX-XXA
Connections:
- net GND: no longer H1.MOUNT, H2.MOUNT, H3.MOUNT, H4.MOUNT
Changed lines of the file:
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@@
 <part name="C43" library="rcl" deviceset="C-EU" device="C0805" value="1u"/>
 <part name="GND69" library="supply1" deviceset="GND" device=""/>
-<part name="H1" library="holes" deviceset="MOUNT-PAD-ROUND" device="3.2"/>
-<part name="H2" library="holes" deviceset="MOUNT-PAD-ROUND" device="3.2"/>
-<part name="H3" library="holes" deviceset="MOUNT-PAD-ROUND" device="3.2"/>
-<part name="H4" library="holes" deviceset="MOUNT-PAD-ROUND" device="3.2"/>
-<part name="GND6" library="supply1" deviceset="GND" device=""/>
 <part name="C4" library="rcl" deviceset="C-EU" device="C0805" value="100n"/>
 <part name="R4" library="rcl" deviceset="R-EU_" device="R0603" value="Rh"/>
@@
 <part name="JP2" library="SparkFun-Connectors" deviceset="M02" device="PTH"/>
 <part name="P+24" library="supply1" deviceset="+5V" device=""/>
+<part name="BOX1" library="hammond" deviceset="HAMMOND-BOX" device="-XXA"/>
 </parts>
 <sheets>
@@
 <wire x1="2.54" y1="200.66" x2="2.54" y2="261.62" width="0.1524" layer="97"/>
 <text x="5.08" y="254" size="5.08" layer="97">CH0</text>
-<wire x1="261.62" y1="10.16" x2="261.62" y2="35.56" width="0.1524" layer="97"/>
-<wire x1="261.62" y1="35.56" x2="281.94" y2="35.56" width="0.1524" layer="97"/>
-<wire x1="281.94" y1="35.56" x2="281.94" y2="10.16" width="0.1524" layer="97"/>
-<wire x1="281.94" y1="10.16" x2="261.62" y2="10.16" width="0.1524" layer="97"/>
 <text x="327.66" y="210.82" size="5.08" layer="97">UART</text>
 <wire x1="325.12" y1="218.44" x2="353.06" y2="218.44" width="0.1524" layer="97"/>
@@
 <instance part="C43" gate="G$1" x="119.38" y="236.22"/>
 <instance part="GND69" gate="1" x="119.38" y="226.06"/>
-<instance part="H1" gate="G$1" x="266.7" y="27.94" smashed="yes" rot="R180">
-<attribute name="NAME" x="266.446" y="32.4358" size="1.778" layer="95" rot="R180"/>
-</instance>
-<instance part="H2" gate="G$1" x="276.86" y="27.94" smashed="yes">
-<attribute name="NAME" x="277.114" y="31.0642" size="1.778" layer="95"/>
-</instance>
-<instance part="H3" gate="G$1" x="266.7" y="20.32" smashed="yes" rot="R180">
-<attribute name="NAME" x="266.446" y="17.1958" size="1.778" layer="95" rot="R180"/>
-</instance>
-<instance part="H4" gate="G$1" x="276.86" y="20.32" smashed="yes">
-<attribute name="NAME" x="277.114" y="17.1958" size="1.778" layer="95" rot="MR180"/>
-</instance>
-<instance part="GND6" gate="1" x="271.78" y="15.24"/>
 <instance part="C4" gate="G$1" x="20.32" y="238.76" smashed="yes">
 <attribute name="NAME" x="22.86" y="236.22" size="1.778" layer="95"/>
@@
 <attribute name="VALUE" x="350.52" y="157.48" size="1.778" layer="96" rot="R180"/>
 </instance>
+<instance part="BOX1" gate="G$1" x="269.24" y="27.94"/>
 </instances>
 <busses>
@@
 </segment>
 <segment>
-<pinref part="H1" gate="G$1" pin="MOUNT"/>
-<pinref part="GND6" gate="1" pin="GND"/>
-<wire x1="269.24" y1="27.94" x2="271.78" y2="27.94" width="0.1524" layer="91"/>
-<pinref part="H4" gate="G$1" pin="MOUNT"/>
-<wire x1="271.78" y1="27.94" x2="271.78" y2="20.32" width="0.1524" layer="91"/>
-<wire x1="271.78" y1="20.32" x2="271.78" y2="17.78" width="0.1524" layer="91"/>
-<wire x1="274.32" y1="20.32" x2="271.78" y2="20.32" width="0.1524" layer="91"/>
-<junction x="271.78" y="20.32"/>
-<pinref part="H3" gate="G$1" pin="MOUNT"/>
-<wire x1="269.24" y1="20.32" x2="271.78" y2="20.32" width="0.1524" layer="91"/>
-<junction x="271.78" y="20.32"/>
-<pinref part="H2" gate="G$1" pin="MOUNT"/>
-<wire x1="274.32" y1="27.94" x2="271.78" y2="27.94" width="0.1524" layer="91"/>
-<junction x="271.78" y="27.94"/>
-</segment>
-<segment>

Commit message: 8x: progress save
Parts:
- removed JP2: (no value), SparkFun-Connectors:M02PTH
- added D9: BAT54C, diode:BAT54C
Connections:
- removed net N$49: IC12.RO, JP2.2
- new net VIN_BUS: D9.A1, U3.4, U3.5
- new net VIN_USB: D9.A2, U$1.VBUS
- net +5V: now also D9.CC; no longer U$1.VBUS, U3.4, U3.5
- net CH0_GAIN: now also IC3.PD5(T1/OC0B/PCINT21); no longer IC3.PB4(MISO/PCINT4), ISP1.1
- net CH1_GAIN: now also IC3.PD6(AIN0/OC0A/PCINT22); no longer IC3.PB5(SCK/PCINT5), ISP1.4
- net CH2_GAIN: now also IC3.PD7(AIN1/PCINT23); no longer IC3.PD5(T1/OC0B/PCINT21)
- net CH3_GAIN: now also IC3.PB0(ICP1/CLKO/PCINT0); no longer IC3.PD6(AIN0/OC0A/PCINT22)
- net CH4_GAIN: now also IC3.PB5(SCK/PCINT5), ISP1.3; no longer IC3.PD7(AIN1/PCINT23)
- net CH5_GAIN: now also IC3.PB4(MISO/PCINT4), ISP1.1; no longer IC3.PB0(ICP1/CLKO/PCINT0)
- net CH6_GAIN: now also IC3.PB2(SS/OC1B/PCINT2); no longer IC3.PB1(OC1A/PCINT1)
- net CH7_GAIN: now also IC3.PB1(OC1A/PCINT1); no longer IC3.PB2(SS/OC1B/PCINT2)
- net LED: now also ISP1.4
- net UART_EN: no longer ISP1.3
- net UART_RX: now also IC12.RO; no longer JP2.1
