File: hardware/usb-current-meter-8x.brd (EAGLE design)
At the start: 94 x 44.5 mm, 154 parts, among them IC10 OPA2234U, IC12 LTC485S, IC2 OPA2234U, IC3 MEGA48/88/168-AU, IC4 OPA2234U, IC5 OPA2234U, IC6 OPA2234U, IC7 OPA2234U, IC8 OPA2234U, IC9 OPA2234U, U3 RJ45-8PTH, X1 MC2, X2 MC2, X3 MC2, X4 MC2, X5 MC2, X6 MC2, X7 MC2, X8 MC2

Commit message: hw: 8x: add part numbers
Parts:
- IC10, IC2, IC4, IC5, IC6, IC7, IC8, IC9: value OPA2234U -> LM358
- IC12: value LTC485S -> MAX3072
- IC3: value MEGA48/88/168-AU -> ATmega168P-20AU
- Y1: value (none) -> 12Mhz
Changed lines of the file:
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@@
 <setting verticaltext="up"/>
 </settings>
-<grid distance="16" unitdist="mil" unit="mil" style="lines" multiple="1" display="yes" altdistance="0.025" altunitdist="inch" altunit="inch"/>
+<grid distance="16" unitdist="mil" unit="mil" style="lines" multiple="1" display="no" altdistance="0.025" altunitdist="inch" altunit="inch"/>
 <layers>
 <layer number="1" name="Top" color="4" fill="1" visible="yes" active="yes"/>
@@
 <element name="ISP1" library="balto" package="2X03" value="" x="69.6976" y="15.0368" rot="R180"/>
 <element name="U$1" library="SparkFun" package="USB-MINIB" value="USB-MINIB-5PIN" x="69.9008" y="5.6896" rot="R90"/>
-<element name="Y1" library="SparkFun" package="HC49U-V" value="" x="53.848" y="5.2832"/>
+<element name="Y1" library="SparkFun" package="HC49U-V" value="12Mhz" x="53.848" y="5.2832"/>
 <element name="C9" library="rcl" package="C0805" value=".1u" x="58.1152" y="22.1488" rot="R90"/>
 <element name="C10" library="rcl" package="C0805" value="22p" x="53.848" y="6.9088" rot="MR0"/>
@@
 <element name="C12" library="rcl" package="C0805" value=".1u" x="56.2864" y="9.9568" rot="MR270"/>
 <element name="C13" library="rcl" package="C0805" value=".1u" x="50.5968" y="9.9568" rot="MR270"/>
-<element name="IC3" library="avr-5" package="TQFP32-08" value="MEGA48/88/168-AU" x="53.0352" y="15.6464" rot="R45"/>
-<element name="IC9" library="burr-brown" package="SO08" value="OPA2234U" x="13.0048" y="26.8224" rot="R180">
+<element name="IC3" library="avr-5" package="TQFP32-08" value="ATmega168P-20AU" x="53.0352" y="15.6464" rot="R45"/>
+<element name="IC9" library="burr-brown" package="SO08" value="LM358" x="13.0048" y="26.8224" rot="R180">
 <attribute name="OC_NEWARK" value="96K4523" x="-14.9352" y="31.9024" size="1.778" layer="27" rot="R180" display="off"/>
 <attribute name="MPN" value="OPA2234U" x="-14.9352" y="31.9024" size="1.778" layer="27" rot="R180" display="off"/>
@@
 <element name="U$2" library="balto" package="CREATIVE_COMMONS" value="Fabio Baltieri" x="8.3312" y="1.2192"/>
 <element name="JP1" library="SparkFun-Connectors" package="1X04" value="" x="43.8912" y="3.6576" rot="R180"/>
-<element name="IC2" library="burr-brown" package="SO08" value="OPA2234U" x="22.7584" y="33.3248" rot="R180">
+<element name="IC2" library="burr-brown" package="SO08" value="LM358" x="22.7584" y="33.3248" rot="R180">
 <attribute name="OC_NEWARK" value="96K4523" x="41.0464" y="21.5392" size="1.778" layer="27" rot="R180" display="off"/>
 <attribute name="MPN" value="OPA2234U" x="41.0464" y="21.5392" size="1.778" layer="27" rot="R180" display="off"/>
@@
 <element name="R11" library="rcl" package="R0603" value="Rh" x="19.5072" y="32.9184" rot="R270"/>
 <element name="C16" library="rcl" package="C0805" value="0" x="19.304" y="29.6672" rot="R90"/>
-<element name="IC4" library="burr-brown" package="SO08" value="OPA2234U" x="32.512" y="33.3248" rot="R180">
+<element name="IC4" library="burr-brown" package="SO08" value="LM358" x="32.512" y="33.3248" rot="R180">
 <attribute name="OC_NEWARK" value="96K4523" x="50.8" y="21.5392" size="1.778" layer="27" rot="R180" display="off"/>
 <attribute name="MPN" value="OPA2234U" x="50.8" y="21.5392" size="1.778" layer="27" rot="R180" display="off"/>
@@
 <element name="R19" library="rcl" package="R0603" value="Rh" x="29.2608" y="32.9184" rot="R270"/>
 <element name="C22" library="rcl" package="C0805" value="0" x="29.0576" y="29.6672" rot="R90"/>
-<element name="IC5" library="burr-brown" package="SO08" value="OPA2234U" x="42.2656" y="33.3248" rot="R180">
+<element name="IC5" library="burr-brown" package="SO08" value="LM358" x="42.2656" y="33.3248" rot="R180">
 <attribute name="OC_NEWARK" value="96K4523" x="60.96" y="21.5392" size="1.778" layer="27" rot="R180" display="off"/>
 <attribute name="MPN" value="OPA2234U" x="60.96" y="21.5392" size="1.778" layer="27" rot="R180" display="off"/>
@@
 <element name="R26" library="rcl" package="R0603" value="Rh" x="39.0144" y="32.9184" rot="R270"/>
 <element name="C28" library="rcl" package="C0805" value="0" x="38.8112" y="29.6672" rot="R90"/>
-<element name="IC6" library="burr-brown" package="SO08" value="OPA2234U" x="52.0192" y="33.3248" rot="R180">
+<element name="IC6" library="burr-brown" package="SO08" value="LM358" x="52.0192" y="33.3248" rot="R180">
 <attribute name="OC_NEWARK" value="96K4523" x="70.7136" y="21.5392" size="1.778" layer="27" rot="R180" display="off"/>
 <attribute name="MPN" value="OPA2234U" x="70.7136" y="21.5392" size="1.778" layer="27" rot="R180" display="off"/>
@@
 <element name="R33" library="rcl" package="R0603" value="Rh" x="48.768" y="32.9184" rot="R270"/>
 <element name="C34" library="rcl" package="C0805" value="0" x="48.5648" y="29.6672" rot="R90"/>
-<element name="IC7" library="burr-brown" package="SO08" value="OPA2234U" x="61.7728" y="33.3248" rot="R180">
+<element name="IC7" library="burr-brown" package="SO08" value="LM358" x="61.7728" y="33.3248" rot="R180">
 <attribute name="OC_NEWARK" value="96K4523" x="80.4672" y="21.5392" size="1.778" layer="27" rot="R180" display="off"/>
 <attribute name="MPN" value="OPA2234U" x="80.4672" y="21.5392" size="1.778" layer="27" rot="R180" display="off"/>
@@
 <element name="R40" library="rcl" package="R0603" value="Rh" x="58.5216" y="32.9184" rot="R270"/>
 <element name="C44" library="rcl" package="C0805" value="0" x="58.3184" y="29.6672" rot="R90"/>
-<element name="IC8" library="burr-brown" package="SO08" value="OPA2234U" x="71.5264" y="33.3248" rot="R180">
+<element name="IC8" library="burr-brown" package="SO08" value="LM358" x="71.5264" y="33.3248" rot="R180">
 <attribute name="OC_NEWARK" value="96K4523" x="90.2208" y="21.1328" size="1.778" layer="27" rot="R180" display="off"/>
 <attribute name="MPN" value="OPA2234U" x="90.2208" y="21.1328" size="1.778" layer="27" rot="R180" display="off"/>
@@
 <element name="R47" library="rcl" package="R0603" value="Rh" x="68.2752" y="32.9184" rot="R270"/>
 <element name="C50" library="rcl" package="C0805" value="0" x="68.072" y="29.6672" rot="R90"/>
-<element name="IC10" library="burr-brown" package="SO08" value="OPA2234U" x="81.28" y="26.8224" rot="R180">
+<element name="IC10" library="burr-brown" package="SO08" value="LM358" x="81.28" y="26.8224" rot="R180">
 <attribute name="OC_NEWARK" value="96K4523" x="99.9744" y="15.0368" size="1.778" layer="27" rot="R180" display="off"/>
 <attribute name="MPN" value="OPA2234U" x="99.9744" y="15.0368" size="1.778" layer="27" rot="R180" display="off"/>
@@
 <element name="R59" library="rcl" package="R0603" value="Rh" x="78.0288" y="26.416" rot="R270"/>
 <element name="C56" library="rcl" package="C0805" value="0" x="77.8256" y="23.1648" rot="R90"/>
-<element name="IC12" library="linear-technology" package="SOIC8" value="LTC485S" x="40.2336" y="11.3792">
+<element name="IC12" library="linear-technology" package="SOIC8" value="MAX3072" x="40.2336" y="11.3792">
 <attribute name="OC_NEWARK" value="unknown" x="40.2336" y="11.3792" size="1.778" layer="27" display="off"/>
 <attribute name="MPN" value="" x="40.2336" y="11.3792" size="1.778" layer="27" display="off"/>
@@
 </signal>
 </signals>
-<errors>
-</errors>
 </board>
 </drawing>
