File: hardware/current-meter-nrf.brd (EAGLE design)
At the start: 44 x 29 mm, 47 parts, among them IC1 TINY24/44/84-SSU, IC2 LM358, IC3 MAX1555, U2 NRF24L01SMD, U3 USB-MINIB-5PIN, X1 MC2, Y1 16M

Commit message: hw: nrf: progress save
Parts:
- removed R1, R2: 68, rcl:R0603
- removed R3: 1k5, rcl:R0603
- moved R13 1.29 mm to (23.6, 19.1)
- moved LED1 1.29 mm to (23.6, 17.5)
Connections:
- removed net N$1: R2.1, R3.1, U3.D-
- removed net N$2: R1.1, U3.D+
- removed net USB_DN: IC1.3, R2.2
- removed net USB_DP: IC1.5, R1.2
- new net LED: IC1.2, LED1.A
- net A_EN: now also IC1.3; no longer IC1.2, LED1.A
- net VCC: no longer R3.2
Routing:
- net USB_DN: track 16.0 -> 0.00 mm, vias 1 -> 0
- net USB_DP: track 15.8 -> 0.00 mm, vias 1 -> 0
- net VCC: track 81.9 -> 70.9 mm
- net LED: track 0.00 -> 5.88 mm
- net N$1: track 5.46 -> 0.00 mm, vias 1 -> 0
- net N$2: track 3.98 -> 0.00 mm, vias 1 -> 0
- net GND: vias 29 -> 30

Commit message: hw: nrf: progress save
Parts:
- removed LED2: (no value), led:SML0805
- removed R10: 330, rcl:R0603
- added C1, C2: 1u, rcl:C0805
- moved TP2 7.72 mm to (11.6, 1.63)
- moved TP1 6.50 mm to (17.3, 1.63)
- moved LED1 2.44 mm to (23.6, 19.9), turned to 180 degrees
- moved R13 0.81 mm to (23.6, 18.3), turned to 0 degrees
- moved C6 0.45 mm to (31.1, 7.92)
- moved C7 0.37 mm to (32.3, 9.14)
- moved L3 0.10 mm to (14.8, 14.9)
- moved C11 0.10 mm to (12.2, 18.8)
- moved C12 0.10 mm to (13.0, 20.8)
- moved C13 0.10 mm to (15.8, 17.0)
- moved C14 0.10 mm to (17.1, 17.0)
- moved TP3 0.05 mm to (11.0, 20.7)
Connections:
- removed net N$20: LED2.C, R10.2
- net +5V: now also C2.1
- net CHG: now also IC1.6; no longer R10.1
- net GND: now also C1.2, C2.2, LED1.C; no longer R13.1
- net LED: now also R13.2; no longer LED1.A
- net N$3: now also LED1.A, R13.1; no longer LED1.C, R13.2
- net RF_IRQ: now also IC1.5; no longer IC1.6
- net VCC: now also C1.1; no longer LED2.A
Routing:
- net +5V: track 8.61 -> 11.4 mm, vias 0 -> 1
- net CHG: track 12.8 -> 15.1 mm, vias 0 -> 2
- net N$20: track 1.55 -> 0.00 mm
- net RF_IRQ: track 12.9 -> 14.3 mm
- net LED: track 5.88 -> 6.61 mm
- net VCC: track 70.9 -> 71.2 mm, vias 4 -> 3
- net GND: vias 30 -> 32

Commit message: hw: nrf: progress save
Parts:
- TP1, TP2: value TPTP11R -> TPTP12R; device testpad:TP11R -> testpad:TP12R
Changed lines of the file:
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@@
 <setting verticaltext="up"/>
 </settings>
-<grid distance="8" unitdist="mil" unit="mil" style="lines" multiple="1" display="yes" altdistance="0.025" altunitdist="inch" altunit="inch"/>
+<grid distance="0.2032" unitdist="mm" unit="mm" style="lines" multiple="1" display="yes" altdistance="0.025" altunitdist="inch" altunit="inch"/>
 <layers>
 <layer number="1" name="Top" color="4" fill="1" visible="yes" active="yes"/>
@@
 <board>
 <plain>
-<hole x="13.4112" y="1.6256" drill="0.8"/>
-<hole x="15.4432" y="1.6256" drill="0.8"/>
+<hole x="13.4112" y="1.8288" drill="1.2"/>
+<hole x="15.4432" y="1.8288" drill="1.2"/>
 <text x="13.8176" y="22.352" size="1.4224" layer="121">FB2012</text>
 <text x="23.5712" y="22.352" size="1.016" layer="121">current-meter-nrf</text>
@@
 <element name="U$1" library="antenna" package="DN007+5" value="INVERTED_F_ANTENNA+5" x="9.9568" y="25.1968"/>
 <element name="IC3" library="maxim" package="SOT23-5L" value="MAX1555" x="27.432" y="3.048"/>
-<element name="TP1" library="testpad" package="TP11R" value="TPTP11R" x="17.272" y="1.6256" rot="MR0">
+<element name="TP1" library="testpad" package="TP12R" value="TPTP12R" x="17.272" y="1.6256" rot="MR0">
 <attribute name="TP_SIGNAL_NAME" value="" x="0.762" y="-54.2544" size="1.778" layer="28" rot="MR0" display="off"/>
 </element>
-<element name="TP2" library="testpad" package="TP11R" value="TPTP11R" x="11.5824" y="1.6256" rot="MR0">
+<element name="TP2" library="testpad" package="TP12R" value="TPTP12R" x="11.5824" y="1.6256" rot="MR0">
 <attribute name="TP_SIGNAL_NAME" value="" x="-10.0076" y="-54.2544" size="1.778" layer="28" rot="MR0" display="off"/>
 </element>
@@
 <wire x1="10.3632" y1="7.112" x2="9.5504" y2="6.2992" width="0.2032" layer="1"/>
 <via x="9.5504" y="6.2992" extent="1-16" drill="0.508"/>
-<wire x1="22.5552" y1="2.6416" x2="13.0048" y2="2.6416" width="0.2032" layer="16"/>
-<wire x1="13.0048" y1="2.6416" x2="9.5504" y2="6.096" width="0.2032" layer="16"/>
+<wire x1="22.5552" y1="2.6416" x2="19.5072" y2="2.6416" width="0.2032" layer="16"/>
+<wire x1="19.5072" y1="2.6416" x2="19.1008" y2="3.048" width="0.2032" layer="16"/>
+<wire x1="19.1008" y1="3.048" x2="12.5984" y2="3.048" width="0.2032" layer="16"/>
+<wire x1="12.5984" y1="3.048" x2="9.5504" y2="6.096" width="0.2032" layer="16"/>
 <wire x1="9.5504" y1="6.096" x2="9.5504" y2="6.2992" width="0.2032" layer="16"/>
 </signal>
@@
 <via x="10.7696" y="6.2992" extent="1-16" drill="0.508"/>
 <wire x1="10.7696" y1="6.2992" x2="10.7696" y2="5.4864" width="0.2032" layer="16"/>
-<wire x1="10.7696" y1="5.4864" x2="13.208" y2="3.048" width="0.2032" layer="16"/>
-<wire x1="13.208" y1="3.048" x2="22.352" y2="3.048" width="0.2032" layer="16"/>
+<wire x1="10.7696" y1="5.4864" x2="12.8016" y2="3.4544" width="0.2032" layer="16"/>
+<wire x1="12.8016" y1="3.4544" x2="19.304" y2="3.4544" width="0.2032" layer="16"/>
+<wire x1="19.304" y1="3.4544" x2="19.7104" y2="3.048" width="0.2032" layer="16"/>
+<wire x1="19.7104" y1="3.048" x2="22.352" y2="3.048" width="0.2032" layer="16"/>
 </signal>
 <signal name="RF_IRQ">

Commit message: nrf: hw: progress save
Parts:
- added C4: .1u, rcl:C0805
- added U4: V_REG_LDOSMD, SparkFun-PowerIC:SOT23-5
- C1, C2: value 1u -> .1u
- C3: value 100n -> .1u
- moved C1 1.93 mm to (25.4, 2.44), flipped to the bottom, turned to 225 degrees
- moved TP2 0.45 mm to (11.2, 1.83)
- moved TP1 0.45 mm to (16.9, 1.83)
- moved IC3 0.41 mm to (27.8, 3.05)
Connections:
- new net VBATT: C4.1, IC3.5, TP1.TP, U4.1, U4.3
- net GND: now also C4.2, U4.2
- net VCC: now also U4.5; no longer IC3.5, TP1.TP
Routing:
- net VBATT: track 0.00 -> 13.3 mm, vias 0 -> 1
- net VCC: track 71.2 -> 66.7 mm
- net MOSI: track 26.6 -> 25.8 mm
- net GND: vias 32 -> 34

Commit message: hw: nrf: add missing part value
Parts:
- C9: value tbd -> 0r
- R5, R6: value tbd -> 10k
- R7: value tbd -> 1k
- R8: value tbd -> 3k3
Changed lines of the file:
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@@
 <element name="C3" library="rcl" package="C0805" value=".1u" x="19.5072" y="16.6624" rot="R90"/>
 <element name="R4" library="rcl" package="R0805" value="Rload" x="42.672" y="16.256" rot="MR270"/>
-<element name="R5" library="rcl" package="R0603" value="tbd" x="41.8592" y="13.4112" rot="MR0"/>
-<element name="R6" library="rcl" package="R0603" value="tbd" x="36.9824" y="13.0048" rot="MR90"/>
-<element name="R7" library="rcl" package="R0603" value="tbd" x="35.7632" y="17.6784" rot="MR0"/>
-<element name="R8" library="rcl" package="R0603" value="tbd" x="32.9184" y="17.6784" rot="MR0"/>
+<element name="R5" library="rcl" package="R0603" value="10k" x="41.8592" y="13.4112" rot="MR0"/>
+<element name="R6" library="rcl" package="R0603" value="10k" x="36.9824" y="13.0048" rot="MR90"/>
+<element name="R7" library="rcl" package="R0603" value="1k" x="35.7632" y="17.6784" rot="MR0"/>
+<element name="R8" library="rcl" package="R0603" value="3k3" x="32.9184" y="17.6784" rot="MR0"/>
 <element name="R12" library="rcl" package="R0603" value="100k" x="31.2928" y="14.224" rot="MR270"/>
 <element name="C6" library="rcl" package="C0805" value="1u" x="31.0896" y="7.9248" rot="R315"/>
@@
 <element name="R13" library="rcl" package="R0603" value="330" x="23.5712" y="18.288"/>
 <element name="ISP1" library="balto" package="2X03" value="" x="3.4544" y="11.9888" rot="R270"/>
-<element name="C9" library="rcl" package="C0805" value="tbd" x="35.7632" y="19.304" rot="MR0"/>
+<element name="C9" library="rcl" package="C0805" value="0r" x="35.7632" y="19.304" rot="MR0"/>
 <element name="C10" library="rcl" package="C0805" value="1u" x="41.0464" y="16.256" rot="MR90"/>
 <element name="C11" library="rcl" package="C0603" value="1p5" x="12.192" y="18.796" rot="R90"/>
@@
 </signal>
 </signals>
-<errors>
-</errors>
 </board>
 </drawing>
